File: Electrical/Main-Board/Main-Board.sch (EAGLE design)
At the start: 0 parts

Commit message: Updated schematic and ignore all backup files
Parts:
- added IC1: ATMEGA16A-PU, SamacSys_Parts:ATMEGA16A-PU
- added J1: FTSH-105-01-L-DV-K-A-P-TR, SamacSys_Parts:FTSH-105-01-L-DV-K-A-P-TR
- added R1: 10K/10%, rcl:R-EU_R0603
- added S1: PTS647SM50SMTR2LFS, SamacSys_Parts:PTS647SM50SMTR2LFS
Connections:
- new net +5V/1: IC1.AREF, IC1.AVCC, IC1.VCC, J1.7, R1.2
- new net GND: IC1.GND, IC1.GND_1, J1.10, J1.6, S1.3, S1.4
- new net RST: IC1.!RESET, J1.8, R1.1, S1.1, S1.2
- new net TCK: IC1.PC2_[TCK], J1.1
- new net TDI: IC1.PC5_[TDI], J1.5
- new net TDO: IC1.PC4_[TDO], J1.2
- new net TMS: IC1.PC3_[TMS], J1.3
- new net TRST: J1.9
