File: Electrical/Main-Board/Main-Board.sch (EAGLE design)
At the start: 41 parts, among them IC1 ATMEGA16A-PU, IC10 TLE4966L, IC2 ATMEGA16A-PU, IC3 AZ1117CH-ADJTRG1, IC4 AZ1117CH-5.0TRG1DITR-ND, IC5 LM2904DRG3, IC6 TLE4966L, IC7 TLE4966L, IC8 TLE4966L, IC9 TLE4966L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

Commit message: Added the final components to the schmatic and updated the layout
Parts:
- removed C7: EEEFK1J220P, SamacSys_Parts:EEEFK1J220P
- removed IC10, IC7, IC8, IC9: TLE4966L, SamacSys_Parts:TLE4966L
- removed IC4: AZ1117CH-5.0TRG1DITR-ND, SamacSys_Parts:AZ1117CH-5.0TRG1DITR-ND
- removed R12, R13, R14, R15, R16: 1.2K/5%, rcl:R-EU_R0603
- removed R5: 200R/5%, rcl:R-EU_R0603
- removed R6: 866R/5%, rcl:R-EU_R0603
- added JP1: (no value), pinhead:PINHD-1X7
- IC3: value AZ1117CH-ADJTRG1 -> TLE4966L; device SamacSys_Parts:AZ1117CH-ADJTRG1 -> SamacSys_Parts:TLE4966L
Connections:
- net +7.5V renamed MOTOR_VCC
- removed net +12V: C7.+, IC3.INPUT, IC4.INPUT, J4.SLEEVE
- removed net DABDA: IC3.OUTPUT, IC3.VOUT, R5.2, R7.1, R8.R1
- removed net LOWER-DISK-LIMIT: IC2.[INT1]_PD3
- removed net UPPER-DISK-LIMIT: IC2.[INT0]_PD2
- removed net W3R355: IC3.ADJ/GND, R5.1, R6.2
- new net HALL_DIR-LOWER: IC2.[INT0]_PD2, IC6.Q1
- new net HALL_DIR-UPPER: IC2.[INT1]_PD3, IC3.Q1
- new net HALL_SPEED-LOWER: IC2.[TXD]_PD1, IC6.Q2
- new net HALL_SPEED-UPPER: IC2.[RXD]_PD0, IC3.Q2
- new net RGB-INT: IC1.[INT0]_PD2, JP1.6
- new net RGB-LED: IC1.[OC1B]_PD4, JP1.7
- net +5V/1: now also IC3.VS, IC6.VS, J4.SLEEVE, JP1.1, R7.1, R8.R1; no longer IC4.OUTPUT, IC4.VOUT_TAB
- net GND: now also IC3.GND, IC6.GND, JP1.2; no longer C7.-, IC4.ADJ/GND, R6.1
- net SCL: now also JP1.4
- net SDA: now also JP1.5
Other:
- note added: "2x16 Alphanumeric display"
- note added: "Current sense"
- note added: "DC input jack"
- note added: "Decoupling capacitors"
- note added: "Hall effect sensors"
- note added: "Programming header"
- note added: "RGB sensor"
- note added: "Servo motor connectors"
- note added: "µC#1 (Master device)"
- note added: "µC#2 (Motor controller)"

Commit message: LCD is wrong, need to finish teh new footprint for it.
Parts:
- added C7: EEEFK1J220P, SamacSys_Parts:EEEFK1J220P
Connections:
- net +5V/1: now also C7.+
- net GND: now also C7.-
Changed lines of the file:
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@@
 <drawing>
 <settings>
-<setting alwaysvectorfont="yes"/>
+<setting alwaysvectorfont="no"/>
 <setting verticaltext="up"/>
 </settings>
@@
 <part name="SUPPLY13" library="supply2" library_urn="urn:adsk.eagle:library:372" deviceset="+5V/1" device=""/>
 <part name="FRAME3" library="frames" library_urn="urn:adsk.eagle:library:229" deviceset="A4L-LOC" device=""/>
+<part name="C7" library="SamacSys_Parts" deviceset="EEEFK1J220P" device=""/>
 </parts>
 <sheets>
@@
 <attribute name="VALUE" x="214.884" y="38.481" size="1.778" layer="96"/>
 </instance>
-<instance part="SUPPLY7" gate="G$1" x="63.5" y="132.08" smashed="yes">
-<attribute name="VALUE" x="60.325" y="135.255" size="1.778" layer="96"/>
+<instance part="SUPPLY7" gate="G$1" x="63.5" y="137.16" smashed="yes">
+<attribute name="VALUE" x="60.325" y="140.335" size="1.778" layer="96"/>
+</instance>
+<instance part="C7" gate="G$1" x="71.12" y="127" smashed="yes" rot="R270">
+<attribute name="NAME" x="72.39" y="128.27" size="1.778" layer="95" align="center-left"/>
+<attribute name="VALUE" x="72.39" y="125.73" size="1.778" layer="96" align="center-left"/>
 </instance>
 </instances>
@@
 </segment>
 <segment>
-<wire x1="63.5" y1="119.38" x2="63.5" y2="104.14" width="0.1524" layer="91"/>
+<wire x1="63.5" y1="119.38" x2="63.5" y2="111.76" width="0.1524" layer="91"/>
 <pinref part="GND12" gate="1" pin="GND"/>
 <pinref part="J4" gate="G$1" pin="TIP"/>
+<wire x1="63.5" y1="111.76" x2="63.5" y2="104.14" width="0.1524" layer="91"/>
 <wire x1="60.96" y1="119.38" x2="63.5" y2="119.38" width="0.1524" layer="91"/>
+<pinref part="C7" gate="G$1" pin="-"/>
+<wire x1="71.12" y1="114.3" x2="71.12" y2="111.76" width="0.1524" layer="91"/>
+<wire x1="71.12" y1="111.76" x2="63.5" y2="111.76" width="0.1524" layer="91"/>
+<junction x="63.5" y="111.76"/>
 </segment>
 <segment>
@@
 <wire x1="63.5" y1="121.92" x2="63.5" y2="129.54" width="0.1524" layer="91"/>
 <pinref part="J4" gate="G$1" pin="SLEEVE"/>
+<wire x1="63.5" y1="129.54" x2="63.5" y2="134.62" width="0.1524" layer="91"/>
 <wire x1="60.96" y1="121.92" x2="63.5" y2="121.92" width="0.1524" layer="91"/>
 <pinref part="SUPPLY7" gate="G$1" pin="+5V/1"/>
+<pinref part="C7" gate="G$1" pin="+"/>
+<wire x1="71.12" y1="127" x2="71.12" y2="129.54" width="0.1524" layer="91"/>
+<wire x1="71.12" y1="129.54" x2="63.5" y2="129.54" width="0.1524" layer="91"/>
+<junction x="63.5" y="129.54"/>
 </segment>
 </net>
